File: PCBs/OSSC/OSSC.sch (KiCad schematic (older format))
At the start: 6 parts, among them J1 Conn_01x02_Female, U1 MCP1700-3302E_SOT23, U2 ESP32-WROOM-32, U3 MPU-6050

Commit message: Schematic Change
-Removed 2 Cap between IC-Ground to Ground
-Added Power-Up Delay-Circuit for ESP
-Added Filter-Cap for MPU
Parts:
- added R1: 10k, Resistor_SMD:R_0603_1608Metric_Pad1.05x0.95mm_HandSolder, symbol OSSC-eagle-import:RESISTOR0402
- C1, C2: value C -> 0.1mu
Connections:
- wire segments 13 -> 18
Other:
- moved on the sheet: C2
Changed lines of the file:
@@
 $EndDescr
-$Comp
-L RF_Module:ESP32-WROOM-32 U2
-U 1 1 5ED2796E
-P 3150 2800
-F 0 "U2" H 3150 4381 50  0000 C CNN
-F 1 "ESP32-WROOM-32" H 3150 4290 50  0000 C CNN
-F 2 "RF_Module:ESP32-WROOM-32" H 3150 1300 50  0001 C CNN
-F 3 "https://www.espressif.com/sites/default/files/documentation/esp32-wroom-32_datasheet_en.pdf" H 2850 2850 50  0001 C CNN
-	1    3150 2800
-	1    0    0    -1
-$EndComp
 $Comp
 L Regulator_Linear:MCP1700-3302E_SOT23 U1
@@
 $EndComp
 Wire Wire Line
-	1750 1400 3150 1400
+	1750 1400 2100 1400
 Connection ~ 3150 1400
 Wire Wire Line
 	5600 2050 5600 1400
-Wire Wire Line
-	5600 1400 3150 1400
-$Comp
-L power:GND #PWR0104
-U 1 1 5ED2E0F5
-P 5500 3750
-F 0 "#PWR0104" H 5500 3500 50  0001 C CNN
-F 1 "GND" H 5505 3577 50  0000 C CNN
-F 2 "" H 5500 3750 50  0001 C CNN
-F 3 "" H 5500 3750 50  0001 C CNN
-	1    5500 3750
-	1    0    0    -1
-$EndComp
-$Comp
-L Device:C C1
-U 1 1 5ED2ED0E
-P 5500 3600
-F 0 "C1" H 5615 3646 50  0000 L CNN
-F 1 "C" H 5615 3555 50  0000 L CNN
-F 2 "Capacitor_SMD:C_0402_1005Metric" H 5538 3450 50  0001 C CNN
-F 3 "~" H 5500 3600 50  0001 C CNN
-	1    5500 3600
-	1    0    0    -1
-$EndComp
 Wire Wire Line
 	4800 2450 4250 2450
@@
 P 5500 2750
 F 0 "U3" H 5500 1961 50  0000 C CNN
-F 1 "MPU-6050" H 5500 1870 50  0000 C CNN
+F 1 "MPU-6050" H 5750 2200 50  0000 C CNN
 F 2 "Sensor_Motion:InvenSense_QFN-24_4x4mm_P0.5mm" H 5500 1950 50  0001 C CNN
 F 3 "https://store.invensense.com/datasheets/invensense/MPU-6050_DataSheet_V3%204.pdf" H 5500 2600 50  0001 C CNN
@@
 	1    0    0    -1
 $EndComp
+Text Label 5600 2050 0    50   ~ 0
+3.3V
+$Comp
+L RF_Module:ESP32-WROOM-32 U2
+U 1 1 5ED2796E
+P 3150 2800
+F 0 "U2" H 3150 4381 50  0000 C CNN
+F 1 "ESP32-WROOM-32" H 2750 4300 50  0000 C CNN
+F 2 "RF_Module:ESP32-WROOM-32" H 3150 1300 50  0001 C CNN
+F 3 "https://www.espressif.com/sites/default/files/documentation/esp32-wroom-32_datasheet_en.pdf" H 2850 2850 50  0001 C CNN
+	1    3150 2800
+	1    0    0    -1
+$EndComp
+Wire Wire Line
+	5600 1400 5450 1400
+$Comp
+L power:GND #PWR0104
+U 1 1 5ED2E0F5
+P 3150 4200
+F 0 "#PWR0104" H 3150 3950 50  0001 C CNN
+F 1 "GND" H 3155 4027 50  0000 C CNN
+F 2 "" H 3150 4200 50  0001 C CNN
+F 3 "" H 3150 4200 50  0001 C CNN
+	1    3150 4200
+	1    0    0    -1
+$EndComp
 $Comp
 L power:GND #PWR01
 U 1 1 5ED353E5
-P 3150 4500
-F 0 "#PWR01" H 3150 4250 50  0001 C CNN
-F 1 "GND" H 3155 4327 50  0000 C CNN
-F 2 "" H 3150 4500 50  0001 C CNN
-F 3 "" H 3150 4500 50  0001 C CNN
-	1    3150 4500
-	1    0    0    -1
+P 5450 1100
+F 0 "#PWR01" H 5450 850 50  0001 C CNN
+F 1 "GND" H 5455 927 50  0000 C CNN
+F 2 "" H 5450 1100 50  0001 C CNN
+F 3 "" H 5450 1100 50  0001 C CNN
+	1    5450 1100
+	-1   0    0    1
 $EndComp
 $Comp
 L Device:C C2
 U 1 1 5ED353EB
-P 3150 4350
-F 0 "C2" H 3265 4396 50  0000 L CNN
-F 1 "C" H 3265 4305 50  0000 L CNN
-F 2 "Capacitor_SMD:C_0402_1005Metric" H 3188 4200 50  0001 C CNN
-F 3 "~" H 3150 4350 50  0001 C CNN
-	1    3150 4350
-	1    0    0    -1
-$EndComp
-Text Label 5600 2050 0    50   ~ 0
-3.3V
+P 5450 1250
+F 0 "C2" H 5565 1296 50  0000 L CNN
+F 1 "0.1mu" H 5565 1205 50  0000 L CNN
+F 2 "Capacitor_SMD:C_0402_1005Metric" H 5488 1100 50  0001 C CNN
+F 3 "~" H 5450 1250 50  0001 C CNN
+	1    5450 1250
+	-1   0    0    1
+$EndComp
+$Comp
+L power:GND #PWR0102
+U 1 1 5EDA47BE
+P 5500 3450
+F 0 "#PWR0102" H 5500 3200 50  0001 C CNN
+F 1 "GND" H 5505 3277 50  0000 C CNN
+F 2 "" H 5500 3450 50  0001 C CNN
+F 3 "" H 5500 3450 50  0001 C CNN
+	1    5500 3450
+	1    0    0    -1
+$EndComp
+$Comp
+L Device:C C1
+U 1 1 5ED8F6BF
+P 2100 1950
+F 0 "C1" H 2215 1996 50  0000 L CNN
+F 1 "0.1mu" H 2215 1905 50  0000 L CNN
+F 2 "Capacitor_SMD:C_0402_1005Metric" H 2138 1800 50  0001 C CNN
+F 3 "~" H 2100 1950 50  0001 C CNN
+	1    2100 1950
+	-1   0    0    1
+$EndComp
+$Comp
+L OSSC-eagle-import:RESISTOR0402 R1
+U 1 1 5ED90842
+P 2100 1600
+F 0 "R1" V 2146 1522 50  0000 R CNN
+F 1 "10k" V 2055 1522 50  0000 R CNN
+F 2 "Resistor_SMD:R_0603_1608Metric_Pad1.05x0.95mm_HandSolder" H 2100 1600 50  0001 C CNN
+F 3 "" H 2100 1600 50  0001 C CNN
+	1    2100 1600
+	0    -1   -1   0
+$EndComp
+Connection ~ 2100 1400
+Wire Wire Line
+	2100 1400 3150 1400
+Wire Wire Line
+	2550 1600 2350 1600
+Wire Wire Line
+	2350 1600 2350 1800
+Wire Wire Line
+	2350 1800 2100 1800
+Connection ~ 2100 1800
+$Comp
+L power:GND #PWR0106
+U 1 1 5ED93DF9
+P 2100 2100
+F 0 "#PWR0106" H 2100 1850 50  0001 C CNN
+F 1 "GND" H 2105 1927 50  0000 C CNN
+F 2 "" H 2100 2100 50  0001 C CNN
+F 3 "" H 2100 2100 50  0001 C CNN
+	1    2100 2100
+	1    0    0    -1
+$EndComp
+Connection ~ 5450 1400
+Wire Wire Line
+	3150 1400 5450 1400
 $EndSCHEMATC

Commit message: Added Components
Added Components for MPU-6050
Added I2C-Connector for Display
Added two Pins for Programming
Parts:
- added C2: 2.2nF, Capacitor_SMD:C_0402_1005Metric, symbol Device:C
- added C4: 2.3nF, Capacitor_SMD:C_0402_1005Metric, symbol Device:C
- added C5: 0.1uF, Capacitor_SMD:C_0402_1005Metric, symbol Device:C
- added J2: Conn_01x04, Connector_PinHeader_1.27mm:PinHeader_1x04_P1.27mm_Vertical, symbol Connector_Generic:Conn_01x04
- added J3, J4: Conn_01x01, Connector_PinHeader_1.00mm:PinHeader_1x01_P1.00mm_Vertical, symbol Connector_Generic:Conn_01x01
- added R2, R3: 10k, Resistor_SMD:R_0402_1005Metric, symbol Device:R
- C1: value 0.1mu -> 0.1uF
- C3: renamed from C2; value 0.1mu -> 0.1uF
Connections:
- net labels added: I2C-SCL, I2C-SDA, MPU-6050-INT, VCC-3.3V
- wire segments 18 -> 14
Other:
- note added: "I2C-Connector for Display"
- moved on the sheet: C3, U1, U3
